Commit message: Created initial URDFs for the robot

File: urdf/rollobot.urdf.xacro (robot description, xacro)
@@ -1,4 +1,5 @@
 <?xml version="1.0"?>
 <robot name="rollobot">
-    <xacro:include filename="rollobot_frame.xacro"/>
+    <xacro:include filename="rollobot_macros.xacro" />
+    <xacro:include filename="rollobot_frame.xacro" />
 </robot>

File: urdf/rollobot_frame.xacro (robot description, xacro)
@@ -1,3 +1,59 @@
 <?xml version="1.0"?>
 <robot name="rollobot">
+    <link name="base_link"></link>
+    <joint name="chassis_joint" type="fixed">
+        <parent link="base_link"/>
+        <child link="chassis"/>
+        <origin xyz="-0.1 0 0"/>
+    </joint>
+    <link name="chassis">
+        <xacro:chassis_config length="0.3" width="0.3" height="0.15">
+            <origin xyz="0.15 0 0.075" rpy="0 0 0"/>
+            <material name="cyan"/>
+        </xacro:chassis_config>
+        <xacro:inertial_box mass="0.5" x="0.3" y="0.3" z="0.15">
+            <origin xyz="0.15 0 0.075" rpy="0 0 0"/>
+        </xacro:inertial_box>
+    </link>
+    <joint name="left_wheel_joint" type="continuous">
+        <parent link="base_link"/>
+        <child link="left_wheel"/>
+        <origin xyz="0 0.175 0" rpy="-${pi/2} 0 0"/>
+        <axis xyz="0 0 1"/>
+    </joint>
+    <link name="left_wheel">
+        <xacro:wheel_config length="0.04" radius="0.05">
+            <material name="blue" />
+        </xacro:wheel_config>
+        <xacro:inertial_cylinder mass="0.1" length="0.04" radius="0.05">
+            <origin xyz="0 0 0" rpy="0 0 0"/>
+        </xacro:inertial_cylinder>
+    </link>
+    <joint name="right_wheel_joint" type="continuous">
+        <parent link="base_link"/>
+        <child link="right_wheel"/>
+        <origin xyz="0 -0.175 0" rpy="${pi/2} 0 0"/>
+        <axis xyz="0 0 -1"/>
+    </joint>
+    <link name="right_wheel">
+        <xacro:wheel_config length="0.04" radius="0.05">
+            <material name="blue" />
+        </xacro:wheel_config>
+        <xacro:inertial_cylinder mass="0.1" length="0.04" radius="0.05">
+            <origin xyz="0 0 0" rpy="0 0 0"/>
+        </xacro:inertial_cylinder>
+    </link>
+    <joint name="caster_wheel_joint" type="fixed">
+        <parent link="chassis"/>
+        <child link="caster_wheel"/>
+        <origin xyz="0.24 0 0" rpy="0 0 0"/>
+    </joint>
+    <link name="caster_wheel">
+        <xacro:caster_config radius="0.05">
+            <material name="white"/>
+        </xacro:caster_config>
+        <xacro:inertial_sphere mass="0.1" radius="0.05">
+            <origin xyz="0 0 0" rpy="0 0 0"/>
+        </xacro:inertial_sphere>
+    </link>
 </robot>

Commit message: Fixed errors in URDFs (didn't include xacro properly)

File: urdf/rollobot.urdf.xacro (robot description, xacro)
@@ -1,4 +1,4 @@
 <?xml version="1.0"?>
-<robot name="rollobot">
+<robot xmlns:xacro="http://www.ros.org/wiki/xacro"  name="robot">
     <xacro:include filename="rollobot_macros.xacro" />
     <xacro:include filename="rollobot_frame.xacro" />

File: urdf/rollobot_frame.xacro (robot description, xacro)
@@ -1,5 +1,6 @@
 <?xml version="1.0"?>
-<robot name="rollobot">
-    <link name="base_link"></link>
+<robot xmlns:xacro="http://www.ros.org/wiki/xacro">
+    <link name="base_link">
+    </link>
     <joint name="chassis_joint" type="fixed">
         <parent link="base_link"/>

File: urdf/rollobot_macros.xacro (robot description, xacro)
@@ -1,4 +1,4 @@
 <?xml version="1.0"?>
-<robot name="rollobot">
+<robot xmlns:xacro="http://www.ros.org/wiki/xacro">
     <!-- Set up colour tags -->
     <material name="white">
@@ -29,9 +29,9 @@
             </geometry>
         </collision>
-    </xacrO:macro>
+    </xacro:macro>
     <xacro:macro name="wheel_config" params="length radius *material">
         <visual>
             <geometry>
-                <cylinder length="${length}" radius="${radius}" />/>
+                <cylinder length="${length}" radius="${radius}" />
             </geometry>
             <xacro:insert_block name="material" />
@@ -39,5 +39,5 @@
         <collision>
             <geometry>
-                <cylinder length="${length}" radius="${radius}" />/>
+                <cylinder length="${length}" radius="${radius}" />
             </geometry>
         </collision>
